File: PICmain/PICmain.brd (EAGLE design)
At the start: 77.8 x 63.8 mm, 20 parts, among them IC2 7805T, J1 PIC_ICSP_6_PIN, U1 PIC16F1778

Commit message: temp
Parts:
- removed IC2: 7805T, adafruit (2):TO220H
- removed U$4: MJ-179PH, akizuki:MJ-179PH
- added IC1: 7805T, linear:TO220H
- added U$3: AE-TC78H653FTG, akizuki:AE-TC78H653FTG
- C3: value 100u -> 104; device rcl:E2,5-6 -> rcl:C025-025X050
- C4: value (none) -> 100u; device rcl:C025-025X050 -> rcl:E2,5-6
- R2, R4: value (none) -> 10k
- U$1: value AE-TC78H653FTG -> MJ-179PH; device akizuki:AE-TC78H653FTG -> akizuki:MJ-179PH
- moved C4 28.0 mm to (58.4, 40.9)
- moved C2 25.2 mm to (45.7, 15.9)
- moved U$1 20.0 mm to (48.5, 5.37), turned to 90 degrees
- moved C3 7.88 mm to (50.5, 40.6)
- moved R2 0.42 mm to (8.95, 57.1)
Connections:
- net N$10 renamed LED6
- net N$11 renamed LED8
- net N$12 renamed SW_RED
- net N$18 renamed LED7
- net N$19 renamed SW_BLUE
- net N$2 renamed LED1
- net N$3 renamed VPP
- net N$4 renamed LED2
- net N$5 renamed PGD
- net N$6 renamed LED3
- net N$7 renamed PGC
- net N$8 renamed LED4
- net N$9 renamed LED5
- removed net DVDD: C1.+, C4.1, R1.2, S1.P, S1.S, U$1.VM@0, U$1.VM@1, U$4.J, U$5.J
- removed net N$1: U$1.OUT1, U$2.P$2
- removed net N$13: U$1.OUT3, U$2.P$3
- removed net N$14: U$1.OUT4, U$2.P$4
- removed net N$15: U$1.OUT2, U$2.P$1
- removed net N$16: R1.1, U$1.STBY
- removed net N$17: IC2.1, S1.O
- removed net VCC: C2.1, C3.+, C5.1, CONNECTOR1.1@0, CONNECTOR1.1@1, CONNECTOR2.1@0, CONNECTOR2.1@1, IC2.3, J1.5, R3.2, U$6.VIN, U1.20
- new net MDVDD: C1.+, C2.1, R1.2, S1.P, S1.S, U$1.J, U$3.VM@0, U$3.VM@1, U$5.J
- new net OUT1: U$2.P$2, U$3.OUT1
- new net OUT2: U$2.P$1, U$3.OUT2
- new net OUT3: U$2.P$3, U$3.OUT3
- new net OUT4: U$2.P$4, U$3.OUT4
- new net STBY: R1.1, U$3.STBY
- new net VDD: C3.1, C4.+, C5.1, CONNECTOR1.1@0, CONNECTOR1.1@1, CONNECTOR2.1@0, CONNECTOR2.1@1, IC1.3, J1.5, R3.2, U$6.VIN, U1.20
- new net VI: IC1.1, S1.O
- net GND: now also C3.2, C4.-, IC1.2, U$1.B, U$1.S, U$3.GND@0, U$3.GND@1, U$3.GND@2; no longer C3.-, C4.2, IC2.2, U$1.GND@0, U$1.GND@1, U$1.GND@2, U$4.B, U$4.S
- net IN1: now also U$3.IN1; no longer U$1.IN1
- net IN2: now also U$3.IN2; no longer U$1.IN2
- net IN3: now also U$3.IN3; no longer U$1.IN3
- net IN4: now also U$3.IN4; no longer U$1.IN4
- net LARGE: now also U$3.LARGE; no longer U$1.LARGE
- net MODE: now also U$3.MODE; no longer U$1.MODE
Routing:
- net VDD: track 0.00 -> 62.6 mm, vias 0 -> 2
- net VCC: track 62.6 -> 0.00 mm, vias 2 -> 0
- net STBY: track 0.00 -> 16.2 mm
- net N$16: track 16.2 -> 0.00 mm
- net VI: track 0.00 -> 11.5 mm
- net N$17: track 11.5 -> 0.00 mm
- net OUT4: track 0.00 -> 5.74 mm
- net OUT3: track 0.00 -> 5.74 mm
- net N$14: track 5.74 -> 0.00 mm
- net N$13: track 5.74 -> 0.00 mm
- net OUT2: track 0.00 -> 5.72 mm
- net OUT1: track 0.00 -> 5.72 mm
- net N$15: track 5.72 -> 0.00 mm
- net N$1: track 5.72 -> 0.00 mm
- added copper zone on layer 16, net MDVDD
- added copper zone on layer 16, net VDD
- removed copper zone on layer 16, net DVDD
- removed copper zone on layer 16, net VCC
